File: board/plc14500/plc14500.kicad_pcb (KiCad board)
At the start: 2 copper layers, 160.1 x 99.9 mm, 169 parts, among them U1 74HC14, U10 MC14500, U11 74HC14, U12 4011, U13 4099, U14 4051, U2 4051, U3 74HC14, U4 NE555, U5 4099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

Commit message: Fix JMP
Parts:
- removed D40: LED 5MM Red, plc14500:LED_3MM
- removed R56: 680R, Resistor_THT:R_Axial_DIN0204_L3.6mm_D1.6mm_P7.62mm_Horizontal
- moved C11 14.2 mm to (139.0, 85.0), turned to 90 degrees
- moved D39 5.20 mm to (144.2, 86.2)
- moved R55 5.20 mm to (145.5, 75.5)
- moved C10 1.04 mm to (120.2, 80.0)
- moved C12 1.04 mm to (135.5, 85.0)
- moved U9 1.03 mm to (124.3, 86.3)
Connections:
- D39 pad A: Net-(D39-PadA) -> JMP
- R54 pad 2: Net-(D39-PadA) -> (no net)
- U10 pad 10: Net-(D40-PadA) -> (no net)
- U10 pad 12: (no net) -> JMP
- U10 pad 9: Net-(D39-PadA) -> (no net)
- U11 pad 3: (no net) -> JMP
- U11 pad 4: (no net) -> Net-(U11-Pad4)
- U7 pad 10: RES -> Net-(U11-Pad4)
Other:
- board text added: "JMP"
- board text removed: "F"
- board text removed: "O"

Commit message: Board routing
Parts:
- added D40: 1N4148, Diode_THT:D_DO-35_SOD27_P7.62mm_Horizontal, F.Cu at (89.2, 66.8)
- added D51: 1N4148, Diode_THT:D_DO-35_SOD27_P7.62mm_Horizontal, F.Cu at (92.7, 66.8)
- R54: value 1K -> 10K
- moved R54 15.2 mm to (96.1, 66.8), turned to 90 degrees
- moved C7 0.47 mm to (103.4, 62.9)
Connections:
- R54 pad 1: RES -> GND
- R54 pad 2: (no net) -> Net-(D40-Pad1)
- U11 pad 3: JMP -> Net-(D40-Pad1)
Routing:
- net GND: track 0.00 -> 860.1 mm, vias 0 -> 36
- net +5V: track 0.00 -> 564.8 mm
- net D6: track 0.00 -> 244.9 mm, vias 0 -> 1
- net RES: track 0.00 -> 243.7 mm
- net A3: track 0.00 -> 236.5 mm
- net D5: track 0.00 -> 224.5 mm, vias 0 -> 5
- net A4: track 0.00 -> 221.3 mm, vias 0 -> 1
- net A7: track 0.00 -> 213.1 mm
- net D7: track 0.00 -> 210.6 mm, vias 0 -> 1
- net D4: track 0.00 -> 207.6 mm, vias 0 -> 3
- net A6: track 0.00 -> 206.9 mm, vias 0 -> 1
- net D0: track 0.00 -> 191.5 mm
- net A5: track 0.00 -> 190.1 mm
- net D1: track 0.00 -> 177.8 mm, vias 0 -> 1
- net D2: track 0.00 -> 169.5 mm, vias 0 -> 2
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- added copper zone on B.Cu, net GND
- added copper zone on F.Cu, net GND
