File: board/plc14500/plc14500.kicad_pcb (KiCad board)
At the start: 2 copper layers, 160.1 x 99.9 mm, 168 parts, among them U1 74HC14, U10 MC14500, U11 74HC14, U12 4011, U13 4099, U14 4051, U2 4051, U3 74HC14, U4 NE555, U5 4099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

Commit message: Update board 3d models
Parts:
- RV1: footprint Potentiometer_THT:Potentiometer_ACP_CA9-H5_Horizontal -> plc14500:HORIZONTAL_POT
- S1, S10, S11, S15, S17, S2, S3, S4, S9: footprint Button_Switch_THT:SW_Tactile_Straight_KSA0Axx1LFTR -> plc14500:SW_Tactile_THT

Commit message: Add schematic in PDF format for easier peruse
Parts:
- C4, C7: value 10uF -> 470uF
- R15: value 680R -> 2K2
- R30, R31: value 680R -> 1K

Commit message: Fix bootloader, add labels to aseembler
Parts:
- R59: value 680R -> 47K
Changed lines of the file:
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@@
     (35 F.Paste user hide)
     (36 B.SilkS user hide)
-    (37 F.SilkS user)
+    (37 F.SilkS user hide)
     (38 B.Mask user hide)
     (39 F.Mask user hide)
@@
       (effects (font (size 1 1) (thickness 0.15)))
     )
-    (fp_text value 680R (at 3.81 1.92) (layer F.Fab)
+    (fp_text value 47K (at 3.81 1.92) (layer F.Fab)
       (effects (font (size 1 1) (thickness 0.15)))
     )

Commit message: First release artifacts
Parts:
- R53: value 1M -> 10K
- R59: value 47K -> 3K3
Other:
- board text added: "K"
- board text added: "Warning! Install Arduino on the opposite side!"
