File: board/plc14500/plc14500.kicad_pcb (KiCad board)
At the start: 2 copper layers, 160.1 x 99.9 mm, 168 parts, among them U1 74HC14, U10 MC14500, U11 74HC14, U12 4011, U13 4099, U14 4051, U2 4051, U3 74HC14, U4 NE555, U5 4099, U6 Arduino Nano, U7 74HC590A, U8 LH5168, U9 NE555

Commit message: Rev_b board
Parts:
- added R22: 47K, Resistor_THT:R_Axial_DIN0204_L3.6mm_D1.6mm_P7.62mm_Horizontal, F.Cu at (144.9, 117.5)
- moved D19 5.07 mm to (144.3, 58.0)
- moved D18 4.84 mm to (139.2, 58.0)
- moved D28 0.12 mm to (149.3, 58.0)
Connections:
- RV1 pad 1: (no net) -> Net-(R15-Pad1)
- RV1 pad 3: Net-(R15-Pad1) -> (no net)
- U11 pad 5: (no net) -> TMR0-TRG
- U11 pad 6: (no net) -> Net-(U11-Pad6)
- U2 pad 3: D -> Net-(R22-Pad1)
- U4 pad 2: TMR0-TRG -> Net-(U11-Pad6)
Routing:
- net Net-(U11-Pad6): track 0.00 -> 194.0 mm, vias 0 -> 7
- net TMR0-TRG: track 58.9 -> 150.5 mm, vias 0 -> 9
- net Net-(R22-Pad1): track 0.00 -> 8.72 mm, vias 0 -> 2
- net D7: track 210.6 -> 216.0 mm
- net Net-(R29-Pad1): track 36.9 -> 41.8 mm
- net /Input/Output/IN3: track 45.9 -> 50.4 mm
- net Net-(D18-PadA): track 16.9 -> 12.6 mm, vias 0 -> 2
- net D: track 88.3 -> 84.1 mm, vias 0 -> 1
- net Net-(C13-Pad2): track 70.7 -> 74.4 mm
- net Net-(R15-Pad1): track 10.4 -> 13.7 mm
- net Net-(D19-PadA): track 11.5 -> 14.1 mm, vias 0 -> 1
- net Net-(S12-Pad5): track 85.0 -> 87.5 mm
- net IN7: track 75.9 -> 74.0 mm
- net W: track 127.7 -> 129.2 mm
- net /Input/Output/IN5: track 46.5 -> 45.6 mm
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Other:
- board text added: "REV.B"
- board text removed: "REV.A"

Commit message: Updates in preparation for rel 1
Parts:
- R12, R13, R14, R16, R17, R18, R19, R20, R21, R23, R24, R25, R27, R28, R29, R32, R33, R34, R35, R36, R37, R38, R39, R40, R41, R42, R43, R44, R45, R46, R47, R48, R49, R5, R52, R55, R57, R58, R6, R60, R61, R62, R63, R64, R65, R66, R67, R7, R8: value 680R -> 820R

Commit message: Small fixes to schema/assembly layout after test assembly
Parts:
- R53: value 10K -> 820R

Commit message: REV.C (#6)
REV.C board updates
Parts:
- removed D50: LED 3MM Red, plc14500:LED_3MM
- removed R67: 820R, Resistor_THT:R_Axial_DIN0204_L3.6mm_D1.6mm_P7.62mm_Horizontal
Connections:
- D41 pad A: Net-(D41-PadA) -> RR
- U10 pad 15: Net-(D41-PadA) -> RR
- U13 pad 1: Net-(D50-PadA) -> (no net)
- U14 pad 4: Net-(D50-PadA) -> RR
Routing:
- net Net-(D50-PadA): track 101.8 -> 0.00 mm, vias 2 -> 0
- net RR: track 0.00 -> 82.2 mm, vias 0 -> 3
- net Net-(D41-PadA): track 43.1 -> 0.00 mm
- net Net-(D50-PadK): track 3.76 -> 0.00 mm
Other:
- board text added: "6"
- board text added: "REV.C"
- board text removed: "REV.B"

Commit message: Convert to kicad7.0
Other:
- net class Default removed
