File: board/plc14500/CPU.sch (KiCad schematic (older format))
At the start: 72 parts, among them U10 MC14500, U3 74HC14, U7 74HC590A, U8 LH5168, U9 NE555

Commit message: Fix JMP
Parts:
- removed D40: LED 5MM Red, plc14500:LED_3MM, symbol SparkFun-LED:LED5MM
- removed R54: 1K, Resistor_THT:R_Axial_DIN0204_L3.6mm_D1.6mm_P7.62mm_Horizontal, symbol Device:R
- removed R56: 680R, Resistor_THT:R_Axial_DIN0204_L3.6mm_D1.6mm_P7.62mm_Horizontal, symbol Device:R
- added U11: 74HC14, Package_DIP:DIP-14_W7.62mm_LongPads, symbol 74xx:74HC14
Connections:
- net RES: no longer U7.10 (~MRC)
- net JMP: now reaches U10.12 (JMP)
- net JMP: now also D39.A, U11.3
- net at U10.9 (FLAGF): no longer D39.A
- new net: U11.4, U7.10 (~MRC)
- no-connect marks 4 -> 5
Other:
- note removed: "*2"
- note removed: "*2) The resistor limits current when there's a bus contention between FLAGF and the onboard reset\nbutton/programmer output"
- moved on the sheet: D39, R55
Changed lines of the file:
@@
 Wire Wire Line
 	2325 3750 2325 3775
-Text GLabel 2000 4250 0    50   Input ~ 0
-RES
+Text GLabel 1300 4250 0    50   Input ~ 0
+JMP
 Wire Wire Line
 	2400 4250 2000 4250
@@
 Wire Wire Line
 	2400 1750 2400 2125
-Text Notes 10800 6500 2    50   ~ 0
-*2) The resistor limits current when there's a bus contention between FLAGF and the onboard reset\nbutton/programmer output
 Text Label 5125 5800 2    50   ~ 0
 D6
@@
 L SparkFun-LED:LED5MM D?
 U 1 1 63B91CBF
-P 9925 4950
+P 10075 4950
 AR Path="/63B91CBF" Ref="D?"  Part="1"
 AR Path="/6394A5B3/63B91CBF" Ref="D39"  Part="1"
-F 0 "D39" H 9950 5025 45  0000 L CNN
-F 1 "LED 5MM Red" H 10003 4911 45  0001 L CNN
-F 2 "plc14500:LED_3MM" V 9725 4950 20  0001 C CNN
-F 3 "" H 9925 4950 50  0001 C CNN
-F 4 "XXX-00000" H 10003 4816 60  0001 L CNN "Field4"
-F 5 "0.01" H 9925 4950 50  0001 C CNN "Price"
-	1    9925 4950
-	1    0    0    -1
-$EndComp
-$Comp
-L SparkFun-LED:LED5MM D?
-U 1 1 63B91CC6
-P 10100 4950
-AR Path="/63B91CC6" Ref="D?"  Part="1"
-AR Path="/6394A5B3/63B91CC6" Ref="D40"  Part="1"
-F 0 "D40" H 10125 5025 45  0000 L CNN
-F 1 "LED 5MM Red" H 10178 4911 45  0001 L CNN
-F 2 "plc14500:LED_3MM" V 9900 4950 20  0001 C CNN
-F 3 "" H 10100 4950 50  0001 C CNN
-F 4 "XXX-00000" H 10178 4816 60  0001 L CNN "Field4"
-F 5 "0.01" H 10100 4950 50  0001 C CNN "Price"
-	1    10100 4950
+F 0 "D39" H 10100 5025 45  0000 L CNN
+F 1 "LED 5MM Red" H 10153 4911 45  0001 L CNN
+F 2 "plc14500:LED_3MM" V 9875 4950 20  0001 C CNN
+F 3 "" H 10075 4950 50  0001 C CNN
+F 4 "XXX-00000" H 10153 4816 60  0001 L CNN "Field4"
+F 5 "0.01" H 10075 4950 50  0001 C CNN "Price"
+	1    10075 4950
 	1    0    0    -1
 $EndComp
@@
 L Device:R R?
 U 1 1 63B91CDA
-P 9925 5400
+P 10075 5400
 AR Path="/63B91CDA" Ref="R?"  Part="1"
 AR Path="/6394A5B3/63B91CDA" Ref="R55"  Part="1"
-F 0 "R55" H 9900 5250 50  0000 R CNN
-F 1 "680R" V 9825 5500 50  0000 R CNN
-F 2 "Resistor_THT:R_Axial_DIN0204_L3.6mm_D1.6mm_P7.62mm_Horizontal" V 9855 5400 50  0001 C CNN
-F 3 "~" H 9925 5400 50  0001 C CNN
-F 4 "0.01" H 9925 5400 50  0001 C CNN "Price"
-	1    9925 5400
-	-1   0    0    1
-$EndComp
-$Comp
-L Device:R R?
-U 1 1 63B91CE0
-P 10100 5400
-AR Path="/63B91CE0" Ref="R?"  Part="1"
-AR Path="/6394A5B3/63B91CE0" Ref="R56"  Part="1"
-F 0 "R56" H 10075 5250 50  0000 R CNN
-F 1 "680R" V 10000 5500 50  0000 R CNN
-F 2 "Resistor_THT:R_Axial_DIN0204_L3.6mm_D1.6mm_P7.62mm_Horizontal" V 10030 5400 50  0001 C CNN
-F 3 "~" H 10100 5400 50  0001 C CNN
-F 4 "0.01" H 10100 5400 50  0001 C CNN "Price"
-	1    10100 5400
+F 0 "R55" H 10050 5250 50  0000 R CNN
+F 1 "680R" V 9975 5500 50  0000 R CNN
+F 2 "Resistor_THT:R_Axial_DIN0204_L3.6mm_D1.6mm_P7.62mm_Horizontal" V 10005 5400 50  0001 C CNN
+F 3 "~" H 10075 5400 50  0001 C CNN
+F 4 "0.01" H 10075 5400 50  0001 C CNN "Price"
+	1    10075 5400
 	-1   0    0    1
 $EndComp
@@
 $EndComp
 Wire Wire Line
-	9925 5150 9925 5250
-Wire Wire Line
-	10100 5150 10100 5250
+	10075 5150 10075 5250
 Wire Wire Line
 	10275 5150 10275 5250
@@
 	10275 5550 10275 5700
 Wire Wire Line
-	10100 5550 10100 5700
-Wire Wire Line
-	9925 5550 9925 5700
-Wire Wire Line
-	9925 4500 9925 4850
-Wire Wire Line
-	10100 4350 9300 4350
-Wire Wire Line
-	10100 4350 10100 4850
+	10075 5550 10075 5700
 Wire Wire Line
 	9300 3900 10275 3900
@@
 	1    0    0    -1
 $EndComp
-Wire Wire Line
-	9925 5700 10100 5700
-Connection ~ 10100 5700
 Connection ~ 10275 5700
 Wire Wire Line
@@
 Wire Wire Line
 	10200 5750 10200 5700
-Wire Wire Line
-	10100 5700 10200 5700
 Connection ~ 10200 5700
 Wire Wire Line
@@
 Processor
 NoConn ~ 9300 4200
-NoConn ~ 9300 4050
+NoConn ~ 9300 4350
 Text GLabel 3750 6950 2    50   Input ~ 0
 WEN
@@
 Wire Wire Line
 	8650 5750 8650 5700
-Text GLabel 9475 5000 2    50   Output ~ 0
-RES
-Wire Wire Line
-	9300 4500 9400 4500
-$Comp
-L Device:R R?
-U 1 1 64EB521E
-P 9400 4725
-AR Path="/64EB521E" Ref="R?"  Part="1"
-AR Path="/6394A5B3/64EB521E" Ref="R54"  Part="1"
-F 0 "R54" H 9375 4575 50  0000 R CNN
-F 1 "1K" V 9300 4825 50  0000 R CNN
-F 2 "Resistor_THT:R_Axial_DIN0204_L3.6mm_D1.6mm_P7.62mm_Horizontal" V 9330 4725 50  0001 C CNN
-F 3 "~" H 9400 4725 50  0001 C CNN
-F 4 "0.01" H 9400 4725 50  0001 C CNN "Price"
-	1    9400 4725
-	-1   0    0    1
-$EndComp
-Wire Wire Line
-	9400 4500 9400 4575
-Connection ~ 9400 4500
-Wire Wire Line
-	9400 4500 9925 4500
-Wire Wire Line
-	9400 4875 9400 5000
-Wire Wire Line
-	9400 5000 9475 5000
-Text Notes 9575 4700 2    50   ~ 0
-*2
 Text Notes 10750 6300 2    50   ~ 0
 *1) Why A13 to one? This allows to use both 32Kx8 and 8Kx8 (that have pin 13 as a second CE)
@@
 	1    0    0    -1
 $EndComp
+Wire Wire Line
+	10075 5700 10200 5700
+NoConn ~ 9300 4500
+Wire Wire Line
+	9300 4050 10075 4050
+Text GLabel 9925 4500 0    50   Output ~ 0
+JMP
+Wire Wire Line
+	10075 4050 10075 4500
+Wire Wire Line
+	9925 4500 10075 4500
+Connection ~ 10075 4500
+Wire Wire Line
+	10075 4500 10075 4850
+$Comp
+L 74xx:74HC14 U?
+U 2 1 637C3E72
+P 1700 4250
+AR Path="/637C3E72" Ref="U?"  Part="1"
+AR Path="/6394A5B3/637C3E72" Ref="U11"  Part="2"
+F 0 "U11" H 1750 4400 50  0000 C CNN
+F 1 "74HC14" H 1550 4050 50  0000 C CNN
+F 2 "Package_DIP:DIP-14_W7.62mm_LongPads" H 1700 4250 50  0001 C CNN
+F 3 "http://www.ti.com/lit/gpn/sn74HC14" H 1700 4250 50  0001 C CNN
+F 4 "0.16" H 1700 4250 50  0001 C CNN "Price"
+	2    1700 4250
+	1    0    0    -1
+$EndComp
+Wire Wire Line
+	1300 4250 1400 4250
 Wire Bus Line
 	7800 3650 7800 4100

Commit message: Board routing
Parts:
- added D40, D51: 1N4148, Diode_THT:D_DO-35_SOD27_P7.62mm_Horizontal, symbol Diode:1N4148
- added R54: 10K, Resistor_THT:R_Axial_DIN0204_L3.6mm_D1.6mm_P7.62mm_Horizontal, symbol Device:R
Connections:
- net GND: now also R54.1
- net JMP: now also D40.2 (A); no longer U11.3
- net RES: now also D51.2 (A)
- new net: D40.1 (K), D51.1 (K), R54.2, U11.3
Changed lines of the file:
@@
 Wire Wire Line
 	2325 3750 2325 3775
-Text GLabel 1300 4250 0    50   Input ~ 0
+Text GLabel 750  4250 0    50   Input ~ 0
 JMP
 Wire Wire Line
@@
 	1    0    0    -1
 $EndComp
-Wire Wire Line
-	1300 4250 1400 4250
+$Comp
+L Diode:1N4148 D40
+U 1 1 637ECCA3
+P 1075 4250
+F 0 "D40" H 1175 4025 50  0000 C CNN
+F 1 "1N4148" H 1075 4124 50  0000 C CNN
+F 2 "Diode_THT:D_DO-35_SOD27_P7.62mm_Horizontal" H 1075 4075 50  0001 C CNN
+F 3 "https://assets.nexperia.com/documents/data-sheet/1N4148_1N4448.pdf" H 1075 4250 50  0001 C CNN
+	1    1075 4250
+	-1   0    0    1
+$EndComp
+$Comp
+L Diode:1N4148 D51
+U 1 1 637EEA46
+P 1075 4425
+F 0 "D51" H 1175 4600 50  0000 C CNN
+F 1 "1N4148" H 1075 4525 50  0000 C CNN
+F 2 "Diode_THT:D_DO-35_SOD27_P7.62mm_Horizontal" H 1075 4250 50  0001 C CNN
+F 3 "https://assets.nexperia.com/documents/data-sheet/1N4148_1N4448.pdf" H 1075 4425 50  0001 C CNN
+	1    1075 4425
+	-1   0    0    1
+$EndComp
+$Comp
+L Device:R R?
+U 1 1 637FFB15
+P 1325 4750
+AR Path="/637FFB15" Ref="R?"  Part="1"
+AR Path="/6394A5B3/637FFB15" Ref="R54"  Part="1"
+F 0 "R54" H 1300 4600 50  0000 R CNN
+F 1 "10K" V 1225 4850 50  0000 R CNN
+F 2 "Resistor_THT:R_Axial_DIN0204_L3.6mm_D1.6mm_P7.62mm_Horizontal" V 1255 4750 50  0001 C CNN
+F 3 "~" H 1325 4750 50  0001 C CNN
+F 4 "0.01" H 1325 4750 50  0001 C CNN "Price"
+	1    1325 4750
+	-1   0    0    1
+$EndComp
+$Comp
+L power:GND #PWR?
+U 1 1 63800447
+P 1325 4975
+AR Path="/63800447" Ref="#PWR?"  Part="1"
+AR Path="/6394A5B3/63800447" Ref="#PWR078"  Part="1"
+F 0 "#PWR078" H 1325 4725 50  0001 C CNN
+F 1 "GND" H 1330 4802 50  0000 C CNN
+F 2 "" H 1325 4975 50  0001 C CNN
+F 3 "" H 1325 4975 50  0001 C CNN
+	1    1325 4975
+	1    0    0    -1
+$EndComp
+Wire Wire Line
+	750  4250 925  4250
+Wire Wire Line
+	1225 4250 1325 4250
+Wire Wire Line
+	1225 4425 1325 4425
+Wire Wire Line
+	1325 4425 1325 4250
+Connection ~ 1325 4250
+Wire Wire Line
+	1325 4250 1400 4250
+Text GLabel 750  4425 0    50   Input ~ 0
+RES
+Wire Wire Line
+	750  4425 925  4425
+Wire Wire Line
+	1325 4600 1325 4425
+Connection ~ 1325 4425
+Wire Wire Line
+	1325 4975 1325 4900
 Wire Bus Line
 	7800 3650 7800 4100

Commit message: Nano board rev-a prod ready
Parts:
- D18, D19, D20, D21, D22, D23, D24, D25, D26, D27, D28, D29, D30, D31, D32, D33, D34, D35, D36, D37, D38, D39, D41, D42: value LED 5MM Red -> LED 3MM Red
Changed lines of the file:
@@
 AR Path="/6394A5B3/6398068B" Ref="D20"  Part="1"
 F 0 "D20" H 4050 4200 45  0000 L CNN
-F 1 "LED 5MM Red" H 4103 4086 45  0001 L CNN
+F 1 "LED 3MM Red" H 4103 4086 45  0001 L CNN
 F 2 "plc14500:LED_3MM" V 3825 4125 20  0001 C CNN
 F 3 "" H 4025 4125 50  0001 C CNN
@@
 AR Path="/6394A5B3/63980692" Ref="D22"  Part="1"
 F 0 "D22" H 4225 4200 45  0000 L CNN
-F 1 "LED 5MM Red" H 4278 4086 45  0001 L CNN
+F 1 "LED 3MM Red" H 4278 4086 45  0001 L CNN
 F 2 "plc14500:LED_3MM" V 4000 4125 20  0001 C CNN
 F 3 "" H 4200 4125 50  0001 C CNN
@@
 AR Path="/6394A5B3/63980699" Ref="D24"  Part="1"
 F 0 "D24" H 4400 4200 45  0000 L CNN
-F 1 "LED 5MM Red" H 4453 4086 45  0001 L CNN
+F 1 "LED 3MM Red" H 4453 4086 45  0001 L CNN
 F 2 "plc14500:LED_3MM" V 4175 4125 20  0001 C CNN
 F 3 "" H 4375 4125 50  0001 C CNN
@@
 AR Path="/6394A5B3/639806A0" Ref="D26"  Part="1"
 F 0 "D26" H 4575 4200 45  0000 L CNN
-F 1 "LED 5MM Red" H 4628 4086 45  0001 L CNN
+F 1 "LED 3MM Red" H 4628 4086 45  0001 L CNN
 F 2 "plc14500:LED_3MM" V 4350 4125 20  0001 C CNN
 F 3 "" H 4550 4125 50  0001 C CNN
@@
 AR Path="/6394A5B3/639806A7" Ref="D29"  Part="1"
 F 0 "D29" H 4750 4200 45  0000 L CNN
-F 1 "LED 5MM Red" H 4803 4086 45  0001 L CNN
+F 1 "LED 3MM Red" H 4803 4086 45  0001 L CNN
 F 2 "plc14500:LED_3MM" V 4525 4125 20  0001 C CNN
 F 3 "" H 4725 4125 50  0001 C CNN
@@
 AR Path="/6394A5B3/639806AE" Ref="D31"  Part="1"
 F 0 "D31" H 4925 4200 45  0000 L CNN
-F 1 "LED 5MM Red" H 4978 4086 45  0001 L CNN
+F 1 "LED 3MM Red" H 4978 4086 45  0001 L CNN
 F 2 "plc14500:LED_3MM" V 4700 4125 20  0001 C CNN
 F 3 "" H 4900 4125 50  0001 C CNN
@@
 AR Path="/6394A5B3/639806B5" Ref="D34"  Part="1"
 F 0 "D34" H 5100 4200 45  0000 L CNN
-F 1 "LED 5MM Red" H 5153 4086 45  0001 L CNN
+F 1 "LED 3MM Red" H 5153 4086 45  0001 L CNN
 F 2 "plc14500:LED_3MM" V 4875 4125 20  0001 C CNN
 F 3 "" H 5075 4125 50  0001 C CNN
@@
 AR Path="/6394A5B3/639806BC" Ref="D36"  Part="1"
 F 0 "D36" H 5275 4200 45  0000 L CNN
-F 1 "LED 5MM Red" H 5328 4086 45  0001 L CNN
+F 1 "LED 3MM Red" H 5328 4086 45  0001 L CNN
 F 2 "plc14500:LED_3MM" V 5050 4125 20  0001 C CNN
 F 3 "" H 5250 4125 50  0001 C CNN
@@
 AR Path="/6394A5B3/6398074E" Ref="D28"  Part="1"
 F 0 "D28" H 4700 1650 45  0000 L CNN
-F 1 "LED 5MM Red" H 4753 1536 45  0001 L CNN
+F 1 "LED 3MM Red" H 4753 1536 45  0001 L CNN
 F 2 "plc14500:LED_3MM" V 4475 1575 20  0001 C CNN
 F 3 "" H 4675 1575 50  0001 C CNN
@@
 AR Path="/6394A5B3/63980763" Ref="D33"  Part="1"
 F 0 "D33" H 5000 1650 45  0000 L CNN
-F 1 "LED 5MM Red" H 5053 1536 45  0001 L CNN
+F 1 "LED 3MM Red" H 5053 1536 45  0001 L CNN
 F 2 "plc14500:LED_3MM" V 4775 1575 20  0001 C CNN
 F 3 "" H 4975 1575 50  0001 C CNN
@@
 AR Path="/6394A5B3/639807EF" Ref="D18"  Part="1"
 F 0 "D18" H 2225 2300 45  0000 L CNN
-F 1 "LED 5MM Red" H 2278 2186 45  0001 L CNN
+F 1 "LED 3MM Red" H 2278 2186 45  0001 L CNN
 F 2 "plc14500:LED_3MM" V 2000 2225 20  0001 C CNN
 F 3 "" H 2200 2225 50  0001 C CNN
@@
 AR Path="/6394A5B3/639807F6" Ref="D19"  Part="1"
 F 0 "D19" H 2425 2300 45  0000 L CNN
-F 1 "LED 5MM Red" H 2478 2186 45  0001 L CNN
+F 1 "LED 3MM Red" H 2478 2186 45  0001 L CNN
 F 2 "plc14500:LED_3MM" V 2200 2225 20  0001 C CNN
 F 3 "" H 2400 2225 50  0001 C CNN
@@
 AR Path="/6394A5B3/63980886" Ref="D35"  Part="1"
 F 0 "D35" H 5150 6000 45  0000 L CNN
-F 1 "LED 5MM Red" H 5203 5886 45  0001 L CNN
+F 1 "LED 3MM Red" H 5203 5886 45  0001 L CNN
 F 2 "plc14500:LED_3MM" V 4925 5925 20  0001 C CNN
 F 3 "" H 5125 5925 50  0001 C CNN
@@
 AR Path="/6394A5B3/6398088D" Ref="D32"  Part="1"
 F 0 "D32" H 4975 6000 45  0000 L CNN
-F 1 "LED 5MM Red" H 5028 5886 45  0001 L CNN
+F 1 "LED 3MM Red" H 5028 5886 45  0001 L CNN
 F 2 "plc14500:LED_3MM" V 4750 5925 20  0001 C CNN
 F 3 "" H 4950 5925 50  0001 C CNN
@@
 AR Path="/6394A5B3/63980894" Ref="D30"  Part="1"
 F 0 "D30" H 4800 6000 45  0000 L CNN
-F 1 "LED 5MM Red" H 4853 5886 45  0001 L CNN
+F 1 "LED 3MM Red" H 4853 5886 45  0001 L CNN
 F 2 "plc14500:LED_3MM" V 4575 5925 20  0001 C CNN
 F 3 "" H 4775 5925 50  0001 C CNN
@@
 AR Path="/6394A5B3/6398089B" Ref="D27"  Part="1"
 F 0 "D27" H 4625 6000 45  0000 L CNN
-F 1 "LED 5MM Red" H 4678 5886 45  0001 L CNN
+F 1 "LED 3MM Red" H 4678 5886 45  0001 L CNN
 F 2 "plc14500:LED_3MM" V 4400 5925 20  0001 C CNN
 F 3 "" H 4600 5925 50  0001 C CNN
@@
 AR Path="/6394A5B3/639808A2" Ref="D25"  Part="1"
 F 0 "D25" H 4450 6000 45  0000 L CNN
-F 1 "LED 5MM Red" H 4503 5886 45  0001 L CNN
+F 1 "LED 3MM Red" H 4503 5886 45  0001 L CNN
 F 2 "plc14500:LED_3MM" V 4225 5925 20  0001 C CNN
 F 3 "" H 4425 5925 50  0001 C CNN
@@
 AR Path="/6394A5B3/639808A9" Ref="D23"  Part="1"
 F 0 "D23" H 4275 6000 45  0000 L CNN
-F 1 "LED 5MM Red" H 4328 5886 45  0001 L CNN
+F 1 "LED 3MM Red" H 4328 5886 45  0001 L CNN
 F 2 "plc14500:LED_3MM" V 4050 5925 20  0001 C CNN
 F 3 "" H 4250 5925 50  0001 C CNN
@@
 AR Path="/6394A5B3/639808B0" Ref="D21"  Part="1"
 F 0 "D21" H 4100 6000 45  0000 L CNN
-F 1 "LED 5MM Red" H 4153 5886 45  0001 L CNN
+F 1 "LED 3MM Red" H 4153 5886 45  0001 L CNN
 F 2 "plc14500:LED_3MM" V 3875 5925 20  0001 C CNN
 F 3 "" H 4075 5925 50  0001 C CNN
@@
 AR Path="/6394A5B3/63B91CBF" Ref="D39"  Part="1"
 F 0 "D39" H 10100 5025 45  0000 L CNN
-F 1 "LED 5MM Red" H 10153 4911 45  0001 L CNN
+F 1 "LED 3MM Red" H 10153 4911 45  0001 L CNN
 F 2 "plc14500:LED_3MM" V 9875 4950 20  0001 C CNN
 F 3 "" H 10075 4950 50  0001 C CNN
@@
 AR Path="/6394A5B3/63B91CCD" Ref="D41"  Part="1"
 F 0 "D41" H 10300 5025 45  0000 L CNN
-F 1 "LED 5MM Red" H 10353 4911 45  0001 L CNN
+F 1 "LED 3MM Red" H 10353 4911 45  0001 L CNN
 F 2 "plc14500:LED_3MM" V 10075 4950 20  0001 C CNN
 F 3 "" H 10275 4950 50  0001 C CNN
@@
 AR Path="/6394A5B3/63B91CD4" Ref="D42"  Part="1"
 F 0 "D42" H 10475 5025 45  0000 L CNN
-F 1 "LED 5MM Red" H 10528 4911 45  0001 L CNN
+F 1 "LED 3MM Red" H 10528 4911 45  0001 L CNN
 F 2 "plc14500:LED_3MM" V 10250 4950 20  0001 C CNN
 F 3 "" H 10450 4950 50  0001 C CNN
@@
 AR Path="/6394A5B3/64D892FF" Ref="D38"  Part="1"
 F 0 "D38" H 7275 2125 45  0000 L CNN
-F 1 "LED 5MM Red" H 7328 2011 45  0001 L CNN
+F 1 "LED 3MM Red" H 7328 2011 45  0001 L CNN
 F 2 "plc14500:LED_3MM" V 7050 2050 20  0001 C CNN
 F 3 "" H 7250 2050 50  0001 C CNN
@@
 AR Path="/6394A5B3/6817902A" Ref="D37"  Part="1"
 F 0 "D37" H 5325 6000 45  0000 L CNN
-F 1 "LED 5MM Red" H 5378 5886 45  0001 L CNN
+F 1 "LED 3MM Red" H 5378 5886 45  0001 L CNN
 F 2 "plc14500:LED_3MM" V 5100 5925 20  0001 C CNN
 F 3 "" H 5300 5925 50  0001 C CNN

Commit message: Update board 3d models
Parts:
- S17: footprint Button_Switch_THT:SW_Tactile_Straight_KSA0Axx1LFTR -> plc14500:SW_Tactile_THT
Changed lines of the file:
@@
 F 0 "S17" V 5371 2277 50  0000 R CNN
 F 1 "Push Button" V 5280 2277 50  0001 R CNN
-F 2 "Button_Switch_THT:SW_Tactile_Straight_KSA0Axx1LFTR" H 5325 2525 50  0001 C CNN
+F 2 "plc14500:SW_Tactile_THT" H 5325 2525 50  0001 C CNN
 F 3 "~" H 5325 2525 50  0001 C CNN
 F 4 "0.01" H 5325 2325 50  0001 C CNN "Price"

Commit message: Add schematic in PDF format for easier peruse
Parts:
- C7: value 10uF -> 470uF
- R30, R31: value 680R -> 1K
Other:
- note added: "Fhi = 1.44 / (R30+2×R31) × C10\nFhi = 4.8KHz\n\nFlo = 1.44 / (R30+2×R31) × (C10+C7)\nFlo = 1Hz"
Changed lines of the file:
@@
 AR Path="/6394A5B3/639805F9" Ref="R31"  Part="1"
 F 0 "R31" H 2700 1300 50  0000 R CNN
-F 1 "680R" H 2700 1375 50  0000 R CNN
+F 1 "1K" H 2700 1375 50  0000 R CNN
 F 2 "Resistor_THT:R_Axial_DIN0204_L3.6mm_D1.6mm_P7.62mm_Horizontal" V 2555 1600 50  0001 C CNN
 F 3 "~" H 2625 1600 50  0001 C CNN
@@
 AR Path="/6394A5B3/639805FF" Ref="R30"  Part="1"
 F 0 "R30" H 2700 1475 50  0000 R CNN
-F 1 "680R" H 2700 1550 50  0000 R CNN
+F 1 "1K" H 2700 1550 50  0000 R CNN
 F 2 "Resistor_THT:R_Axial_DIN0204_L3.6mm_D1.6mm_P7.62mm_Horizontal" V 2380 1600 50  0001 C CNN
 F 3 "~" H 2450 1600 50  0001 C CNN
@@
 P 1325 2525
 F 0 "C7" H 1443 2571 50  0000 L CNN
-F 1 "10uF" H 1443 2480 50  0000 L CNN
+F 1 "470uF" H 1443 2480 50  0000 L CNN
 F 2 "Capacitor_THT:CP_Radial_D8.0mm_P5.00mm" H 1363 2375 50  0001 C CNN
 F 3 "~" H 1325 2525 50  0001 C CNN
@@
 Wire Bus Line
 	3475 3800 3475 4975
+Text Notes 750  3250 0    50   ~ 0
+Fhi = 1.44 / (R30+2×R31) × C10\nFhi = 4.8KHz\n\nFlo = 1.44 / (R30+2×R31) × (C10+C7)\nFlo = 1Hz
 $EndSCHEMATC

Commit message: First release artifacts
Parts:
- R53: value 1M -> 10K
Changed lines of the file:
@@
 AR Path="/6394A5B3/63980939" Ref="R53"  Part="1"
 F 0 "R53" V 7693 5050 50  0000 C CNN
-F 1 "1M" V 7784 5050 50  0000 C CNN
+F 1 "10K" V 7784 5050 50  0000 C CNN
 F 2 "Resistor_THT:R_Axial_DIN0204_L3.6mm_D1.6mm_P7.62mm_Horizontal" V 7830 5050 50  0001 C CNN
 F 3 "~" H 7900 5050 50  0001 C CNN
