File: board/plc14500/CPU.sch (KiCad schematic (older format))
At the start: 73 parts, among them U10 MC14500, U11 74HC14, U3 74HC14, U7 74HC590A, U8 LH5168, U9 NE555

Commit message: Updates in preparation for rel 1
Parts:
- R28, R29, R32, R33, R34, R35, R36, R37, R38, R39, R40, R41, R42, R43, R44, R45, R46, R47, R48, R49, R52, R55, R57, R58: value 680R -> 820R
Changed lines of the file:
@@
 AR Path="/6394A5B3/639806CA" Ref="R32"  Part="1"
 F 0 "R32" H 4000 4425 50  0000 R CNN
-F 1 "680R" V 3925 4675 50  0000 R CNN
+F 1 "820R" V 3925 4675 50  0000 R CNN
 F 2 "Resistor_THT:R_Axial_DIN0204_L3.6mm_D1.6mm_P7.62mm_Horizontal" V 3955 4575 50  0001 C CNN
 F 3 "~" H 4025 4575 50  0001 C CNN
@@
 AR Path="/6394A5B3/639806D0" Ref="R34"  Part="1"
 F 0 "R34" H 4175 4425 50  0000 R CNN
-F 1 "680R" V 4100 4675 50  0000 R CNN
+F 1 "820R" V 4100 4675 50  0000 R CNN
 F 2 "Resistor_THT:R_Axial_DIN0204_L3.6mm_D1.6mm_P7.62mm_Horizontal" V 4130 4575 50  0001 C CNN
 F 3 "~" H 4200 4575 50  0001 C CNN
@@
 AR Path="/6394A5B3/639806D6" Ref="R36"  Part="1"
 F 0 "R36" H 4350 4425 50  0000 R CNN
-F 1 "680R" V 4275 4675 50  0000 R CNN
+F 1 "820R" V 4275 4675 50  0000 R CNN
 F 2 "Resistor_THT:R_Axial_DIN0204_L3.6mm_D1.6mm_P7.62mm_Horizontal" V 4305 4575 50  0001 C CNN
 F 3 "~" H 4375 4575 50  0001 C CNN
@@
 AR Path="/6394A5B3/639806DC" Ref="R38"  Part="1"
 F 0 "R38" H 4525 4425 50  0000 R CNN
-F 1 "680R" V 4450 4675 50  0000 R CNN
+F 1 "820R" V 4450 4675 50  0000 R CNN
 F 2 "Resistor_THT:R_Axial_DIN0204_L3.6mm_D1.6mm_P7.62mm_Horizontal" V 4480 4575 50  0001 C CNN
 F 3 "~" H 4550 4575 50  0001 C CNN
@@
 AR Path="/6394A5B3/639806E2" Ref="R41"  Part="1"
 F 0 "R41" H 4700 4425 50  0000 R CNN
-F 1 "680R" V 4625 4675 50  0000 R CNN
+F 1 "820R" V 4625 4675 50  0000 R CNN
 F 2 "Resistor_THT:R_Axial_DIN0204_L3.6mm_D1.6mm_P7.62mm_Horizontal" V 4655 4575 50  0001 C CNN
 F 3 "~" H 4725 4575 50  0001 C CNN
@@
 AR Path="/6394A5B3/639806E8" Ref="R43"  Part="1"
 F 0 "R43" H 4875 4425 50  0000 R CNN
-F 1 "680R" V 4800 4675 50  0000 R CNN
+F 1 "820R" V 4800 4675 50  0000 R CNN
 F 2 "Resistor_THT:R_Axial_DIN0204_L3.6mm_D1.6mm_P7.62mm_Horizontal" V 4830 4575 50  0001 C CNN
 F 3 "~" H 4900 4575 50  0001 C CNN
@@
 AR Path="/6394A5B3/639806EE" Ref="R46"  Part="1"
 F 0 "R46" H 5050 4425 50  0000 R CNN
-F 1 "680R" V 4975 4675 50  0000 R CNN
+F 1 "820R" V 4975 4675 50  0000 R CNN
 F 2 "Resistor_THT:R_Axial_DIN0204_L3.6mm_D1.6mm_P7.62mm_Horizontal" V 5005 4575 50  0001 C CNN
 F 3 "~" H 5075 4575 50  0001 C CNN
@@
 AR Path="/6394A5B3/639806F4" Ref="R48"  Part="1"
 F 0 "R48" H 5225 4425 50  0000 R CNN
-F 1 "680R" V 5150 4675 50  0000 R CNN
+F 1 "820R" V 5150 4675 50  0000 R CNN
 F 2 "Resistor_THT:R_Axial_DIN0204_L3.6mm_D1.6mm_P7.62mm_Horizontal" V 5180 4575 50  0001 C CNN
 F 3 "~" H 5250 4575 50  0001 C CNN
@@
 AR Path="/6394A5B3/63980754" Ref="R40"  Part="1"
 F 0 "R40" H 4650 1850 50  0000 R CNN
-F 1 "680R" V 4575 2100 50  0000 R CNN
+F 1 "820R" V 4575 2100 50  0000 R CNN
 F 2 "Resistor_THT:R_Axial_DIN0204_L3.6mm_D1.6mm_P7.62mm_Horizontal" V 4605 2000 50  0001 C CNN
 F 3 "~" H 4675 2000 50  0001 C CNN
@@
 AR Path="/6394A5B3/63980769" Ref="R45"  Part="1"
 F 0 "R45" H 4950 1850 50  0000 R CNN
-F 1 "680R" V 4875 2100 50  0000 R CNN
+F 1 "820R" V 4875 2100 50  0000 R CNN
 F 2 "Resistor_THT:R_Axial_DIN0204_L3.6mm_D1.6mm_P7.62mm_Horizontal" V 4905 2000 50  0001 C CNN
 F 3 "~" H 4975 2000 50  0001 C CNN
@@
 AR Path="/6394A5B3/63980802" Ref="R29"  Part="1"
 F 0 "R29" V 2125 1875 50  0000 C CNN
-F 1 "680R" V 2125 2075 50  0000 C CNN
+F 1 "820R" V 2125 2075 50  0000 C CNN
 F 2 "Resistor_THT:R_Axial_DIN0204_L3.6mm_D1.6mm_P7.62mm_Horizontal" V 1980 1950 50  0001 C CNN
 F 3 "~" H 2050 1950 50  0001 C CNN
@@
 AR Path="/6394A5B3/6398085B" Ref="R47"  Part="1"
 F 0 "R47" H 5100 6225 50  0000 R CNN
-F 1 "680R" V 5025 6475 50  0000 R CNN
+F 1 "820R" V 5025 6475 50  0000 R CNN
 F 2 "Resistor_THT:R_Axial_DIN0204_L3.6mm_D1.6mm_P7.62mm_Horizontal" V 5055 6375 50  0001 C CNN
 F 3 "~" H 5125 6375 50  0001 C CNN
@@
 AR Path="/6394A5B3/63980861" Ref="R44"  Part="1"
 F 0 "R44" H 4925 6225 50  0000 R CNN
-F 1 "680R" V 4850 6475 50  0000 R CNN
+F 1 "820R" V 4850 6475 50  0000 R CNN
 F 2 "Resistor_THT:R_Axial_DIN0204_L3.6mm_D1.6mm_P7.62mm_Horizontal" V 4880 6375 50  0001 C CNN
 F 3 "~" H 4950 6375 50  0001 C CNN
@@
 AR Path="/6394A5B3/63980867" Ref="R42"  Part="1"
 F 0 "R42" H 4750 6225 50  0000 R CNN
-F 1 "680R" V 4675 6475 50  0000 R CNN
+F 1 "820R" V 4675 6475 50  0000 R CNN
 F 2 "Resistor_THT:R_Axial_DIN0204_L3.6mm_D1.6mm_P7.62mm_Horizontal" V 4705 6375 50  0001 C CNN
 F 3 "~" H 4775 6375 50  0001 C CNN
@@
 AR Path="/6394A5B3/6398086D" Ref="R39"  Part="1"
 F 0 "R39" H 4575 6225 50  0000 R CNN
-F 1 "680R" V 4500 6475 50  0000 R CNN
+F 1 "820R" V 4500 6475 50  0000 R CNN
 F 2 "Resistor_THT:R_Axial_DIN0204_L3.6mm_D1.6mm_P7.62mm_Horizontal" V 4530 6375 50  0001 C CNN
 F 3 "~" H 4600 6375 50  0001 C CNN
@@
 AR Path="/6394A5B3/63980873" Ref="R37"  Part="1"
 F 0 "R37" H 4400 6225 50  0000 R CNN
-F 1 "680R" V 4325 6475 50  0000 R CNN
+F 1 "820R" V 4325 6475 50  0000 R CNN
 F 2 "Resistor_THT:R_Axial_DIN0204_L3.6mm_D1.6mm_P7.62mm_Horizontal" V 4355 6375 50  0001 C CNN
 F 3 "~" H 4425 6375 50  0001 C CNN
@@
 AR Path="/6394A5B3/63980879" Ref="R35"  Part="1"
 F 0 "R35" H 4225 6225 50  0000 R CNN
-F 1 "680R" V 4150 6475 50  0000 R CNN
+F 1 "820R" V 4150 6475 50  0000 R CNN
 F 2 "Resistor_THT:R_Axial_DIN0204_L3.6mm_D1.6mm_P7.62mm_Horizontal" V 4180 6375 50  0001 C CNN
 F 3 "~" H 4250 6375 50  0001 C CNN
@@
 AR Path="/6394A5B3/6398087F" Ref="R33"  Part="1"
 F 0 "R33" H 4050 6225 50  0000 R CNN
-F 1 "680R" V 3975 6475 50  0000 R CNN
+F 1 "820R" V 3975 6475 50  0000 R CNN
 F 2 "Resistor_THT:R_Axial_DIN0204_L3.6mm_D1.6mm_P7.62mm_Horizontal" V 4005 6375 50  0001 C CNN
 F 3 "~" H 4075 6375 50  0001 C CNN
@@
 AR Path="/6394A5B3/63B91CDA" Ref="R55"  Part="1"
 F 0 "R55" H 10050 5250 50  0000 R CNN
-F 1 "680R" V 9975 5500 50  0000 R CNN
+F 1 "820R" V 9975 5500 50  0000 R CNN
 F 2 "Resistor_THT:R_Axial_DIN0204_L3.6mm_D1.6mm_P7.62mm_Horizontal" V 10005 5400 50  0001 C CNN
 F 3 "~" H 10075 5400 50  0001 C CNN
@@
 AR Path="/6394A5B3/63B91CE6" Ref="R57"  Part="1"
 F 0 "R57" H 10250 5250 50  0000 R CNN
-F 1 "680R" V 10175 5500 50  0000 R CNN
+F 1 "820R" V 10175 5500 50  0000 R CNN
 F 2 "Resistor_THT:R_Axial_DIN0204_L3.6mm_D1.6mm_P7.62mm_Horizontal" V 10205 5400 50  0001 C CNN
 F 3 "~" H 10275 5400 50  0001 C CNN
@@
 AR Path="/6394A5B3/63B91CEC" Ref="R58"  Part="1"
 F 0 "R58" H 10425 5250 50  0000 R CNN
-F 1 "680R" V 10350 5500 50  0000 R CNN
+F 1 "820R" V 10350 5500 50  0000 R CNN
 F 2 "Resistor_THT:R_Axial_DIN0204_L3.6mm_D1.6mm_P7.62mm_Horizontal" V 10380 5400 50  0001 C CNN
 F 3 "~" H 10450 5400 50  0001 C CNN
@@
 AR Path="/6394A5B3/64D8A141" Ref="R52"  Part="1"
 F 0 "R52" H 7225 2275 50  0000 R CNN
-F 1 "680R" V 7150 2525 50  0000 R CNN
+F 1 "820R" V 7150 2525 50  0000 R CNN
 F 2 "Resistor_THT:R_Axial_DIN0204_L3.6mm_D1.6mm_P7.62mm_Horizontal" V 7180 2425 50  0001 C CNN
 F 3 "~" H 7250 2425 50  0001 C CNN
@@
 AR Path="/6394A5B3/639807FC" Ref="R28"  Part="1"
 F 0 "R28" V 2125 1725 50  0000 R CNN
-F 1 "680R" V 2125 1950 50  0000 R CNN
+F 1 "820R" V 2125 1950 50  0000 R CNN
 F 2 "Resistor_THT:R_Axial_DIN0204_L3.6mm_D1.6mm_P7.62mm_Horizontal" V 1980 1750 50  0001 C CNN
 F 3 "~" H 2050 1750 50  0001 C CNN
@@
 AR Path="/6394A5B3/68179590" Ref="R49"  Part="1"
 F 0 "R49" H 5275 6225 50  0000 R CNN
-F 1 "680R" V 5200 6475 50  0000 R CNN
+F 1 "820R" V 5200 6475 50  0000 R CNN
 F 2 "Resistor_THT:R_Axial_DIN0204_L3.6mm_D1.6mm_P7.62mm_Horizontal" V 5230 6375 50  0001 C CNN
 F 3 "~" H 5300 6375 50  0001 C CNN
