File: board/plc14500/CPU.sch (KiCad schematic (older format))
At the start: 73 parts, among them U10 MC14500, U11 74HC14, U3 74HC14, U7 74HC590A, U8 LH5168, U9 NE555

Commit message: Small fixes to schema/assembly layout after test assembly
Parts:
- R53: value 10K -> 820R
Changed lines of the file:
@@
 AR Path="/6394A5B3/63980939" Ref="R53"  Part="1"
 F 0 "R53" V 7693 5050 50  0000 C CNN
-F 1 "10K" V 7784 5050 50  0000 C CNN
+F 1 "820R" V 7784 5050 50  0000 C CNN
 F 2 "Resistor_THT:R_Axial_DIN0204_L3.6mm_D1.6mm_P7.62mm_Horizontal" V 7830 5050 50  0001 C CNN
 F 3 "~" H 7900 5050 50  0001 C CNN

Commit message: Rescue some missing symbols that were broken
Parts:
- D18, D19, D20, D21, D22, D23, D24, D25, D26, D27, D28, D29, D30, D31, D32, D33, D34, D35, D36, D37, D38, D39, D41, D42: symbol SparkFun-LED:LED5MM -> plc14500-rescue:LED5MM-SparkFun-LED
- S16, S18: symbol SparkFun-Switches:SWITCH-DPDT-PTH-GPI-152-3013 -> plc14500-rescue:SWITCH-DPDT-PTH-GPI-152-3013-SparkFun-Switches
- U9: symbol SparkFun-IC-Special-Function:555D -> plc14500-rescue:555D-SparkFun-IC-Special-Function
Changed lines of the file:
@@
 $EndComp
 $Comp
-L SparkFun-IC-Special-Function:555D U?
+L plc14500-rescue:555D-SparkFun-IC-Special-Function U?
 U 1 1 63980606
 P 3325 1750
@@
 	2800 3425 2800 3375
 $Comp
-L SparkFun-LED:LED5MM D?
+L plc14500-rescue:LED5MM-SparkFun-LED D?
 U 1 1 6398068B
 P 4025 4125
@@
 $EndComp
 $Comp
-L SparkFun-LED:LED5MM D?
+L plc14500-rescue:LED5MM-SparkFun-LED D?
 U 1 1 63980692
 P 4200 4125
@@
 $EndComp
 $Comp
-L SparkFun-LED:LED5MM D?
+L plc14500-rescue:LED5MM-SparkFun-LED D?
 U 1 1 63980699
 P 4375 4125
@@
 $EndComp
 $Comp
-L SparkFun-LED:LED5MM D?
+L plc14500-rescue:LED5MM-SparkFun-LED D?
 U 1 1 639806A0
 P 4550 4125
@@
 $EndComp
 $Comp
-L SparkFun-LED:LED5MM D?
+L plc14500-rescue:LED5MM-SparkFun-LED D?
 U 1 1 639806A7
 P 4725 4125
@@
 $EndComp
 $Comp
-L SparkFun-LED:LED5MM D?
+L plc14500-rescue:LED5MM-SparkFun-LED D?
 U 1 1 639806AE
 P 4900 4125
@@
 $EndComp
 $Comp
-L SparkFun-LED:LED5MM D?
+L plc14500-rescue:LED5MM-SparkFun-LED D?
 U 1 1 639806B5
 P 5075 4125
@@
 $EndComp
 $Comp
-L SparkFun-LED:LED5MM D?
+L plc14500-rescue:LED5MM-SparkFun-LED D?
 U 1 1 639806BC
 P 5250 4125
@@
 	4325 2675 4325 2375
 $Comp
-L SparkFun-Switches:SWITCH-DPDT-PTH-GPI-152-3013 S?
+L plc14500-rescue:SWITCH-DPDT-PTH-GPI-152-3013-SparkFun-Switches S?
 U 1 1 63980747
 P 6800 1700
@@
 $EndComp
 $Comp
-L SparkFun-LED:LED5MM D?
+L plc14500-rescue:LED5MM-SparkFun-LED D?
 U 1 1 6398074E
 P 4675 1575
@@
 	4675 2150 4675 2675
 $Comp
-L SparkFun-LED:LED5MM D?
+L plc14500-rescue:LED5MM-SparkFun-LED D?
 U 1 1 63980763
 P 4975 1575
@@
 	7050 1500 7050 1100
 $Comp
-L SparkFun-Switches:SWITCH-DPDT-PTH-GPI-152-3013 S?
+L plc14500-rescue:SWITCH-DPDT-PTH-GPI-152-3013-SparkFun-Switches S?
 U 1 1 639807D9
 P 1675 1950
@@
 NoConn ~ 1875 2250
 $Comp
-L SparkFun-LED:LED5MM D?
+L plc14500-rescue:LED5MM-SparkFun-LED D?
 U 1 1 639807EF
 P 2200 2225
@@
 $EndComp
 $Comp
-L SparkFun-LED:LED5MM D?
+L plc14500-rescue:LED5MM-SparkFun-LED D?
 U 1 1 639807F6
 P 2400 2225
@@
 $EndComp
 $Comp
-L SparkFun-LED:LED5MM D?
+L plc14500-rescue:LED5MM-SparkFun-LED D?
 U 1 1 63980886
 P 5125 5925
@@
 $EndComp
 $Comp
-L SparkFun-LED:LED5MM D?
+L plc14500-rescue:LED5MM-SparkFun-LED D?
 U 1 1 6398088D
 P 4950 5925
@@
 $EndComp
 $Comp
-L SparkFun-LED:LED5MM D?
+L plc14500-rescue:LED5MM-SparkFun-LED D?
 U 1 1 63980894
 P 4775 5925
@@
 $EndComp
 $Comp
-L SparkFun-LED:LED5MM D?
+L plc14500-rescue:LED5MM-SparkFun-LED D?
 U 1 1 6398089B
 P 4600 5925
@@
 $EndComp
 $Comp
-L SparkFun-LED:LED5MM D?
+L plc14500-rescue:LED5MM-SparkFun-LED D?
 U 1 1 639808A2
 P 4425 5925
@@
 $EndComp
 $Comp
-L SparkFun-LED:LED5MM D?
+L plc14500-rescue:LED5MM-SparkFun-LED D?
 U 1 1 639808A9
 P 4250 5925
@@
 $EndComp
 $Comp
-L SparkFun-LED:LED5MM D?
+L plc14500-rescue:LED5MM-SparkFun-LED D?
 U 1 1 639808B0
 P 4075 5925
@@
 DATA
 $Comp
-L SparkFun-LED:LED5MM D?
+L plc14500-rescue:LED5MM-SparkFun-LED D?
 U 1 1 63B91CBF
 P 10075 4950
@@
 $EndComp
 $Comp
-L SparkFun-LED:LED5MM D?
+L plc14500-rescue:LED5MM-SparkFun-LED D?
 U 1 1 63B91CCD
 P 10275 4950
@@
 $EndComp
 $Comp
-L SparkFun-LED:LED5MM D?
+L plc14500-rescue:LED5MM-SparkFun-LED D?
 U 1 1 63B91CD4
 P 10450 4950
@@
 	2925 7350 2925 7400
 $Comp
-L SparkFun-LED:LED5MM D?
+L plc14500-rescue:LED5MM-SparkFun-LED D?
 U 1 1 64D892FF
 P 7250 2050
@@
 	5700 6550 5925 6550
 $Comp
-L SparkFun-LED:LED5MM D?
+L plc14500-rescue:LED5MM-SparkFun-LED D?
 U 1 1 6817902A
 P 5300 5925

Commit message: REV.C (#6)
REV.C board updates
Connections:
- net RR: now reaches D41.A, U10.15 (RR)
Changed lines of the file:
@@
 Sheet 3 4
 Title "PLC14500 - Nano"
-Date "2022-11-09"
-Rev "0.4"
+Date "2023-03-04"
+Rev "0.5"
 Comp "Nicola Cimmino"
-Comment1 ""
+Comment1 "REV.C"
 Comment2 ""
 Comment3 ""
@@
 Wire Bus Line
 	6025 5600 6150 5600
-$Comp
-L Device:CP C7
-U 1 1 63766840
-P 1325 2525
-F 0 "C7" H 1443 2571 50  0000 L CNN
-F 1 "470uF" H 1443 2480 50  0000 L CNN
-F 2 "Capacitor_THT:CP_Radial_D8.0mm_P5.00mm" H 1363 2375 50  0001 C CNN
-F 3 "~" H 1325 2525 50  0001 C CNN
-	1    1325 2525
-	1    0    0    -1
-$EndComp
 Wire Wire Line
 	10075 5700 10200 5700
@@
 Text Notes 750  3250 0    50   ~ 0
 Fhi = 1.44 / (R30+2×R31) × C10\nFhi = 4.8KHz\n\nFlo = 1.44 / (R30+2×R31) × (C10+C7)\nFlo = 1Hz
+Text GLabel 10550 3900 2    50   Output ~ 0
+RR
+Wire Wire Line
+	10275 3900 10550 3900
+Connection ~ 10275 3900
 Wire Bus Line
 	7800 3650 7800 4100
@@
 Wire Bus Line
 	3475 3800 3475 4975
+$Comp
+L Device:CP C7
+U 1 1 63766840
+P 1325 2525
+F 0 "C7" H 1443 2571 50  0000 L CNN
+F 1 "470uF" H 1443 2480 50  0000 L CNN
+F 2 "Capacitor_THT:CP_Radial_D8.0mm_P5.00mm" H 1363 2375 50  0001 C CNN
+F 3 "~" H 1325 2525 50  0001 C CNN
+	1    1325 2525
+	1    0    0    -1
+$EndComp
 $EndSCHEMATC
