File: board/plc14500/IO.sch (KiCad schematic (older format))
At the start: 71 parts, among them U1 74HC14, U11 74HC14, U2 4051, U3 74HC14, U4 NE555, U5 4099, U6 Arduino Nano

Commit message: REV.C (#6)
REV.C board updates
Parts:
- C4: value 470uF -> 10uF
- RV1: value 10K -> 1M
Other:
- note added: "T= 0.02-11s\nT = 1.1 * C4 * (RV1+R15)"
- note removed: "T= 1-7s\nT = 1.1 * C4 * (RV1+R15)"
Changed lines of the file:
@@
 Title "PLC14500 - Nano"
 Date "2022-11-09"
-Rev "0.4"
+Rev "0.5"
 Comp "Nicola Cimmino"
-Comment1 ""
+Comment1 "REV.C"
 Comment2 ""
 Comment3 ""
@@
 P 6800 4700
 F 0 "RV1" H 6731 4746 50  0000 R CNN
-F 1 "10K" H 6731 4655 50  0000 R CNN
+F 1 "1M" H 6731 4655 50  0000 R CNN
 F 2 "plc14500:HORIZONTAL_POT" H 6800 4700 50  0001 C CNN
 F 3 "~" H 6800 4700 50  0001 C CNN
@@
 AR Path="/63B4BDA9/6376CD92" Ref="C4"  Part="1"
 F 0 "C4" H 6618 6146 50  0000 L CNN
-F 1 "470uF" H 6618 6055 50  0000 L CNN
+F 1 "10uF" H 6618 6055 50  0000 L CNN
 F 2 "Capacitor_THT:CP_Radial_D8.0mm_P5.00mm" H 6538 5950 50  0001 C CNN
 F 3 "~" H 6500 6100 50  0001 C CNN
@@
 $EndComp
 Text Notes 7575 5075 0    50   ~ 0
-T= 1-7s\nT = 1.1 * C4 * (RV1+R15)
+T= 0.02-11s\nT = 1.1 * C4 * (RV1+R15)
 $Comp
 L 74xx:74HC14 U?
