File: board/plc14500/SPRAM.sch (KiCad schematic (older format))
At the start: 25 parts, among them U11 74HC14, U12 4011, U13 4099, U14 4051, U3 74HC14

Commit message: Nano board rev-a prod ready
Parts:
- D43, D44, D45, D46, D47, D48, D49, D50: value LED 5MM Red -> LED 3MM Red
Changed lines of the file:
@@
 AR Path="/67425B3B/674297C9" Ref="D43"  Part="1"
 F 0 "D43" H 7500 3475 45  0000 L CNN
-F 1 "LED 5MM Red" H 7578 3611 45  0001 L CNN
+F 1 "LED 3MM Red" H 7578 3611 45  0001 L CNN
 F 2 "plc14500:LED_3MM" V 7300 3650 20  0001 C CNN
 F 3 "" H 7500 3650 50  0001 C CNN
@@
 AR Path="/67425B3B/674297D0" Ref="D44"  Part="1"
 F 0 "D44" H 7675 3475 45  0000 L CNN
-F 1 "LED 5MM Red" H 7753 3611 45  0001 L CNN
+F 1 "LED 3MM Red" H 7753 3611 45  0001 L CNN
 F 2 "plc14500:LED_3MM" V 7475 3650 20  0001 C CNN
 F 3 "" H 7675 3650 50  0001 C CNN
@@
 AR Path="/67425B3B/674297D7" Ref="D45"  Part="1"
 F 0 "D45" H 7850 3475 45  0000 L CNN
-F 1 "LED 5MM Red" H 7928 3611 45  0001 L CNN
+F 1 "LED 3MM Red" H 7928 3611 45  0001 L CNN
 F 2 "plc14500:LED_3MM" V 7650 3650 20  0001 C CNN
 F 3 "" H 7850 3650 50  0001 C CNN
@@
 AR Path="/67425B3B/674297DE" Ref="D46"  Part="1"
 F 0 "D46" H 8025 3475 45  0000 L CNN
-F 1 "LED 5MM Red" H 8103 3611 45  0001 L CNN
+F 1 "LED 3MM Red" H 8103 3611 45  0001 L CNN
 F 2 "plc14500:LED_3MM" V 7825 3650 20  0001 C CNN
 F 3 "" H 8025 3650 50  0001 C CNN
@@
 AR Path="/67425B3B/674297E5" Ref="D47"  Part="1"
 F 0 "D47" H 8200 3475 45  0000 L CNN
-F 1 "LED 5MM Red" H 8278 3611 45  0001 L CNN
+F 1 "LED 3MM Red" H 8278 3611 45  0001 L CNN
 F 2 "plc14500:LED_3MM" V 8000 3650 20  0001 C CNN
 F 3 "" H 8200 3650 50  0001 C CNN
@@
 AR Path="/67425B3B/674297EC" Ref="D48"  Part="1"
 F 0 "D48" H 8375 3475 45  0000 L CNN
-F 1 "LED 5MM Red" H 8453 3611 45  0001 L CNN
+F 1 "LED 3MM Red" H 8453 3611 45  0001 L CNN
 F 2 "plc14500:LED_3MM" V 8175 3650 20  0001 C CNN
 F 3 "" H 8375 3650 50  0001 C CNN
@@
 AR Path="/67425B3B/674297F3" Ref="D49"  Part="1"
 F 0 "D49" H 8550 3475 45  0000 L CNN
-F 1 "LED 5MM Red" H 8628 3611 45  0001 L CNN
+F 1 "LED 3MM Red" H 8628 3611 45  0001 L CNN
 F 2 "plc14500:LED_3MM" V 8350 3650 20  0001 C CNN
 F 3 "" H 8550 3650 50  0001 C CNN
@@
 AR Path="/67425B3B/67429845" Ref="D50"  Part="1"
 F 0 "D50" H 8725 3475 45  0000 L CNN
-F 1 "LED 5MM Red" H 8803 3611 45  0001 L CNN
+F 1 "LED 3MM Red" H 8803 3611 45  0001 L CNN
 F 2 "plc14500:LED_3MM" V 8525 3650 20  0001 C CNN
 F 3 "" H 8725 3650 50  0001 C CNN

Commit message: Fix bootloader, add labels to aseembler
Parts:
- R59: value 680R -> 47K
Other:
- note added: "Write Outputs"
- note removed: "Write Inputs"
Changed lines of the file:
@@
 AR Path="/67425B3B/67AF2AD4" Ref="R59"  Part="1"
 F 0 "R59" H 1450 3225 50  0000 R CNN
-F 1 "680R" V 1375 3475 50  0000 R CNN
+F 1 "47K" V 1375 3475 50  0000 R CNN
 F 2 "Resistor_THT:R_Axial_DIN0204_L3.6mm_D1.6mm_P7.62mm_Horizontal" V 1405 3375 50  0001 C CNN
 F 3 "~" H 1475 3375 50  0001 C CNN
@@
 Text Notes 4275 6075 2    50   ~ 0
 Write Scratchpad RAM
-Text Notes 3900 6200 2    50   ~ 0
-Write Inputs
+Text Notes 3950 6200 2    50   ~ 0
+Write Outputs
 Text Notes 8775 2100 2    89   ~ 0
 Scratchpad RAM

Commit message: First release artifacts
Parts:
- R59: value 47K -> 3K3
Changed lines of the file:
@@
 AR Path="/67425B3B/67AF2AD4" Ref="R59"  Part="1"
 F 0 "R59" H 1450 3225 50  0000 R CNN
-F 1 "47K" V 1375 3475 50  0000 R CNN
+F 1 "3K3" V 1375 3475 50  0000 R CNN
 F 2 "Resistor_THT:R_Axial_DIN0204_L3.6mm_D1.6mm_P7.62mm_Horizontal" V 1405 3375 50  0001 C CNN
 F 3 "~" H 1475 3375 50  0001 C CNN

Commit message: Updates in preparation for rel 1
Parts:
- R60, R61, R62, R63, R64, R65, R66, R67: value 680R -> 820R
Changed lines of the file:
@@
 AR Path="/67425B3B/674297F9" Ref="R60"  Part="1"
 F 0 "R60" H 7475 3950 50  0000 R CNN
-F 1 "680R" V 7400 4200 50  0000 R CNN
+F 1 "820R" V 7400 4200 50  0000 R CNN
 F 2 "Resistor_THT:R_Axial_DIN0204_L3.6mm_D1.6mm_P7.62mm_Horizontal" V 7430 4100 50  0001 C CNN
 F 3 "~" H 7500 4100 50  0001 C CNN
@@
 AR Path="/67425B3B/674297FF" Ref="R61"  Part="1"
 F 0 "R61" H 7650 3950 50  0000 R CNN
-F 1 "680R" V 7575 4200 50  0000 R CNN
+F 1 "820R" V 7575 4200 50  0000 R CNN
 F 2 "Resistor_THT:R_Axial_DIN0204_L3.6mm_D1.6mm_P7.62mm_Horizontal" V 7605 4100 50  0001 C CNN
 F 3 "~" H 7675 4100 50  0001 C CNN
@@
 AR Path="/67425B3B/67429805" Ref="R62"  Part="1"
 F 0 "R62" H 7825 3950 50  0000 R CNN
-F 1 "680R" V 7750 4200 50  0000 R CNN
+F 1 "820R" V 7750 4200 50  0000 R CNN
 F 2 "Resistor_THT:R_Axial_DIN0204_L3.6mm_D1.6mm_P7.62mm_Horizontal" V 7780 4100 50  0001 C CNN
 F 3 "~" H 7850 4100 50  0001 C CNN
@@
 AR Path="/67425B3B/6742980B" Ref="R63"  Part="1"
 F 0 "R63" H 8000 3950 50  0000 R CNN
-F 1 "680R" V 7925 4200 50  0000 R CNN
+F 1 "820R" V 7925 4200 50  0000 R CNN
 F 2 "Resistor_THT:R_Axial_DIN0204_L3.6mm_D1.6mm_P7.62mm_Horizontal" V 7955 4100 50  0001 C CNN
 F 3 "~" H 8025 4100 50  0001 C CNN
@@
 AR Path="/67425B3B/67429811" Ref="R64"  Part="1"
 F 0 "R64" H 8175 3950 50  0000 R CNN
-F 1 "680R" V 8100 4200 50  0000 R CNN
+F 1 "820R" V 8100 4200 50  0000 R CNN
 F 2 "Resistor_THT:R_Axial_DIN0204_L3.6mm_D1.6mm_P7.62mm_Horizontal" V 8130 4100 50  0001 C CNN
 F 3 "~" H 8200 4100 50  0001 C CNN
@@
 AR Path="/67425B3B/67429817" Ref="R65"  Part="1"
 F 0 "R65" H 8350 3950 50  0000 R CNN
-F 1 "680R" V 8275 4200 50  0000 R CNN
+F 1 "820R" V 8275 4200 50  0000 R CNN
 F 2 "Resistor_THT:R_Axial_DIN0204_L3.6mm_D1.6mm_P7.62mm_Horizontal" V 8305 4100 50  0001 C CNN
 F 3 "~" H 8375 4100 50  0001 C CNN
@@
 AR Path="/67425B3B/6742981D" Ref="R66"  Part="1"
 F 0 "R66" H 8525 3950 50  0000 R CNN
-F 1 "680R" V 8450 4200 50  0000 R CNN
+F 1 "820R" V 8450 4200 50  0000 R CNN
 F 2 "Resistor_THT:R_Axial_DIN0204_L3.6mm_D1.6mm_P7.62mm_Horizontal" V 8480 4100 50  0001 C CNN
 F 3 "~" H 8550 4100 50  0001 C CNN
@@
 AR Path="/67425B3B/6742984B" Ref="R67"  Part="1"
 F 0 "R67" H 8700 3950 50  0000 R CNN
-F 1 "680R" V 8625 4200 50  0000 R CNN
+F 1 "820R" V 8625 4200 50  0000 R CNN
 F 2 "Resistor_THT:R_Axial_DIN0204_L3.6mm_D1.6mm_P7.62mm_Horizontal" V 8655 4100 50  0001 C CNN
 F 3 "~" H 8725 4100 50  0001 C CNN

Commit message: Rescue some missing symbols that were broken
Parts:
- D43, D44, D45, D46, D47, D48, D49, D50: symbol SparkFun-LED:LED5MM -> plc14500-rescue:LED5MM-SparkFun-LED
Changed lines of the file:
@@
 $EndDescr
 $Comp
-L SparkFun-LED:LED5MM D?
+L plc14500-rescue:LED5MM-SparkFun-LED D?
 U 1 1 674297C9
 P 7500 3650
 AR Path="/63B4BDA9/674297C9" Ref="D?"  Part="1"
 AR Path="/67425B3B/674297C9" Ref="D43"  Part="1"
+AR Path="/674297C9" Ref="D43"  Part="1"
 F 0 "D43" H 7500 3475 45  0000 L CNN
 F 1 "LED 3MM Red" H 7578 3611 45  0001 L CNN
@@
 $EndComp
 $Comp
-L SparkFun-LED:LED5MM D?
+L plc14500-rescue:LED5MM-SparkFun-LED D?
 U 1 1 674297D0
 P 7675 3650
 AR Path="/63B4BDA9/674297D0" Ref="D?"  Part="1"
 AR Path="/67425B3B/674297D0" Ref="D44"  Part="1"
+AR Path="/674297D0" Ref="D44"  Part="1"
 F 0 "D44" H 7675 3475 45  0000 L CNN
 F 1 "LED 3MM Red" H 7753 3611 45  0001 L CNN
@@
 $EndComp
 $Comp
-L SparkFun-LED:LED5MM D?
+L plc14500-rescue:LED5MM-SparkFun-LED D?
 U 1 1 674297D7
 P 7850 3650
 AR Path="/63B4BDA9/674297D7" Ref="D?"  Part="1"
 AR Path="/67425B3B/674297D7" Ref="D45"  Part="1"
+AR Path="/674297D7" Ref="D45"  Part="1"
 F 0 "D45" H 7850 3475 45  0000 L CNN
 F 1 "LED 3MM Red" H 7928 3611 45  0001 L CNN
@@
 $EndComp
 $Comp
-L SparkFun-LED:LED5MM D?
+L plc14500-rescue:LED5MM-SparkFun-LED D?
 U 1 1 674297DE
 P 8025 3650
 AR Path="/63B4BDA9/674297DE" Ref="D?"  Part="1"
 AR Path="/67425B3B/674297DE" Ref="D46"  Part="1"
+AR Path="/674297DE" Ref="D46"  Part="1"
 F 0 "D46" H 8025 3475 45  0000 L CNN
 F 1 "LED 3MM Red" H 8103 3611 45  0001 L CNN
@@
 $EndComp
 $Comp
-L SparkFun-LED:LED5MM D?
+L plc14500-rescue:LED5MM-SparkFun-LED D?
 U 1 1 674297E5
 P 8200 3650
 AR Path="/63B4BDA9/674297E5" Ref="D?"  Part="1"
 AR Path="/67425B3B/674297E5" Ref="D47"  Part="1"
+AR Path="/674297E5" Ref="D47"  Part="1"
 F 0 "D47" H 8200 3475 45  0000 L CNN
 F 1 "LED 3MM Red" H 8278 3611 45  0001 L CNN
@@
 $EndComp
 $Comp
-L SparkFun-LED:LED5MM D?
+L plc14500-rescue:LED5MM-SparkFun-LED D?
 U 1 1 674297EC
 P 8375 3650
 AR Path="/63B4BDA9/674297EC" Ref="D?"  Part="1"
 AR Path="/67425B3B/674297EC" Ref="D48"  Part="1"
+AR Path="/674297EC" Ref="D48"  Part="1"
 F 0 "D48" H 8375 3475 45  0000 L CNN
 F 1 "LED 3MM Red" H 8453 3611 45  0001 L CNN
@@
 $EndComp
 $Comp
-L SparkFun-LED:LED5MM D?
+L plc14500-rescue:LED5MM-SparkFun-LED D?
 U 1 1 674297F3
 P 8550 3650
 AR Path="/63B4BDA9/674297F3" Ref="D?"  Part="1"
 AR Path="/67425B3B/674297F3" Ref="D49"  Part="1"
+AR Path="/674297F3" Ref="D49"  Part="1"
 F 0 "D49" H 8550 3475 45  0000 L CNN
 F 1 "LED 3MM Red" H 8628 3611 45  0001 L CNN
@@
 	7675 4400 7850 4400
 $Comp
-L SparkFun-LED:LED5MM D?
+L plc14500-rescue:LED5MM-SparkFun-LED D?
 U 1 1 67429845
 P 8725 3650
 AR Path="/63B4BDA9/67429845" Ref="D?"  Part="1"
 AR Path="/67425B3B/67429845" Ref="D50"  Part="1"
+AR Path="/67429845" Ref="D50"  Part="1"
 F 0 "D50" H 8725 3475 45  0000 L CNN
 F 1 "LED 3MM Red" H 8803 3611 45  0001 L CNN

Commit message: REV.C (#6)
REV.C board updates
Parts:
- removed D50: LED 3MM Red, plc14500:LED_3MM, symbol plc14500-rescue:LED5MM-SparkFun-LED
- removed R67: 820R, Resistor_THT:R_Axial_DIN0204_L3.6mm_D1.6mm_P7.62mm_Horizontal, symbol Device:R
Connections:
- net at U13.1 (Q7): no longer U14.4 (X7)
- new net RR: U14.4 (X7)
- no-connect marks 0 -> 1
Other:
- note added: "*1"
- note added: "*1) Prior to REV.C this was a generic SPR \nand connected to Q7 of U13"
Changed lines of the file:
@@
 Title "Scratchpad RAM"
 Date "2022-11-09"
-Rev "0.4"
+Rev "0.5"
 Comp ""
-Comment1 ""
+Comment1 "REV.C"
 Comment2 ""
 Comment3 ""
@@
 Wire Wire Line
 	7675 4400 7850 4400
-$Comp
-L plc14500-rescue:LED5MM-SparkFun-LED D?
-U 1 1 67429845
-P 8725 3650
-AR Path="/63B4BDA9/67429845" Ref="D?"  Part="1"
-AR Path="/67425B3B/67429845" Ref="D50"  Part="1"
-AR Path="/67429845" Ref="D50"  Part="1"
-F 0 "D50" H 8725 3475 45  0000 L CNN
-F 1 "LED 3MM Red" H 8803 3611 45  0001 L CNN
-F 2 "plc14500:LED_3MM" V 8525 3650 20  0001 C CNN
-F 3 "" H 8725 3650 50  0001 C CNN
-F 4 "XXX-00000" H 8803 3516 60  0001 L CNN "Field4"
-F 5 "0.01" H 8725 3650 50  0001 C CNN "Price"
-	1    8725 3650
-	1    0    0    -1
-$EndComp
-$Comp
-L Device:R R?
-U 1 1 6742984B
-P 8725 4100
-AR Path="/63B4BDA9/6742984B" Ref="R?"  Part="1"
-AR Path="/67425B3B/6742984B" Ref="R67"  Part="1"
-F 0 "R67" H 8700 3950 50  0000 R CNN
-F 1 "820R" V 8625 4200 50  0000 R CNN
-F 2 "Resistor_THT:R_Axial_DIN0204_L3.6mm_D1.6mm_P7.62mm_Horizontal" V 8655 4100 50  0001 C CNN
-F 3 "~" H 8725 4100 50  0001 C CNN
-F 4 "0.01" H 8725 4100 50  0001 C CNN "Price"
-	1    8725 4100
-	-1   0    0    1
-$EndComp
-Wire Wire Line
-	8550 4400 8725 4400
-Wire Wire Line
-	8725 4400 8725 4250
-Connection ~ 8550 4400
-Wire Wire Line
-	8725 3950 8725 3850
 Wire Wire Line
 	6400 3050 6250 3050
@@
 	7150 3100 8375 3100
 Wire Wire Line
-	7150 3300 8725 3300
-Wire Wire Line
 	7500 3550 7500 2600
 Wire Wire Line
@@
 Wire Wire Line
 	8550 3200 9525 3200
-Wire Wire Line
-	8725 3550 8725 3300
-Connection ~ 8725 3300
-Wire Wire Line
-	8725 3300 9525 3300
 Wire Wire Line
 	9525 3600 9400 3600
@@
 	1    0    0    -1
 $EndComp
+Text GLabel 9350 3300 0    50   Input ~ 0
+RR
+Wire Wire Line
+	9350 3300 9525 3300
+NoConn ~ 7150 3300
 Wire Bus Line
 	9300 3700 9300 4100
 Wire Bus Line
 	6150 3150 6150 4150
+Text Notes 9075 3350 0    50   ~ 0
+*1
+Text Notes 9000 4725 0    50   ~ 0
+*1) Prior to REV.C this was a generic SPR \nand connected to Q7 of U13
 $EndSCHEMATC
